File: hardware/mainboard/AudioIO.sch (KiCad schematic (older format))
At the start: 21 parts, among them J3 AUDIO_IN_L, J4 AUDIO_IN_R, J5 AUDIO_OUT_L, J6 AUDIO_OUT_R, U4 TL074

Commit message: hardware: update schematics & add BOM
Parts:
- J3: value AUDIO_IN_L -> PJ398SM
- J4: value AUDIO_IN_R -> PJ398SM
- J5: value AUDIO_OUT_L -> PJ398SM
- J6: value AUDIO_OUT_R -> PJ398SM
- R14, R15, R6, R7: value 24k -> 10k
Other:
- note added: "Audio In L\n"
- note added: "Audio In R\n"
- note added: "Audio Out L\n"
- note added: "Audio Out R"
Changed lines of the file:
@@
 AR Path="/61C2C7F7/61C471BA" Ref="R14"  Part="1"
 F 0 "R14" V 5850 1700 50  0000 C CNN
-F 1 "24k" V 5950 1700 50  0000 C CNN
+F 1 "10k" V 5950 1700 50  0000 C CNN
 F 2 "Resistor_SMD:R_0603_1608Metric_Pad0.98x0.95mm_HandSolder" V 5680 1700 50  0001 C CNN
 F 3 "" H 5750 1700 50  0001 C CNN
@@
 AR Path="/61C2C7F7/61C471DD" Ref="R15"  Part="1"
 F 0 "R15" V 5850 3050 50  0000 C CNN
-F 1 "24k" V 5950 3050 50  0000 C CNN
+F 1 "10k" V 5950 3050 50  0000 C CNN
 F 2 "Resistor_SMD:R_0603_1608Metric_Pad0.98x0.95mm_HandSolder" V 5680 3050 50  0001 C CNN
 F 3 "" H 5750 3050 50  0001 C CNN
@@
 AR Path="/61C2C7F7/61C471F4" Ref="R6"  Part="1"
 F 0 "R6" V 4150 4050 50  0000 C CNN
-F 1 "24k" V 4250 4050 50  0000 C CNN
+F 1 "10k" V 4250 4050 50  0000 C CNN
 F 2 "Resistor_SMD:R_0603_1608Metric_Pad0.98x0.95mm_HandSolder" V 3980 4050 50  0001 C CNN
 F 3 "" H 4050 4050 50  0001 C CNN
@@
 AR Path="/61C2C7F7/61C47217" Ref="R7"  Part="1"
 F 0 "R7" V 4150 5350 50  0000 C CNN
-F 1 "24k" V 4250 5350 50  0000 C CNN
+F 1 "10k" V 4250 5350 50  0000 C CNN
 F 2 "Resistor_SMD:R_0603_1608Metric_Pad0.98x0.95mm_HandSolder" V 3980 5350 50  0001 C CNN
 F 3 "" H 4050 5350 50  0001 C CNN
@@
 AR Path="/61C2C7F7/61C47250" Ref="J3"  Part="1"
 F 0 "J3" H 3622 1584 50  0000 R CNN
-F 1 "AUDIO_IN_L" H 3622 1675 50  0000 R CNN
+F 1 "PJ398SM" H 3622 1675 50  0000 R CNN
 F 2 "ell_connectors:THONKICONN" H 4083 1883 50  0001 C CNN
 F 3 "" H 4200 1400 50  0000 C CNN
@@
 AR Path="/61C2C7F7/61C47260" Ref="J4"  Part="1"
 F 0 "J4" H 3622 2934 50  0000 R CNN
-F 1 "AUDIO_IN_R" H 3622 3025 50  0000 R CNN
+F 1 "PJ398SM" H 3622 3025 50  0000 R CNN
 F 2 "ell_connectors:THONKICONN" H 4083 3233 50  0001 C CNN
 F 3 "" H 4200 2750 50  0000 C CNN
@@
 AR Path="/61C2C7F7/61C47270" Ref="J5"  Part="1"
 F 0 "J5" H 5522 4034 50  0000 R CNN
-F 1 "AUDIO_OUT_L" H 5522 4125 50  0000 R CNN
+F 1 "PJ398SM" H 5522 4125 50  0000 R CNN
 F 2 "ell_connectors:THONKICONN" H 5983 4333 50  0001 C CNN
 F 3 "" H 6100 3850 50  0000 C CNN
@@
 AR Path="/61C2C7F7/61C47280" Ref="J6"  Part="1"
 F 0 "J6" H 5522 5334 50  0000 R CNN
-F 1 "AUDIO_OUT_R" H 5522 5425 50  0000 R CNN
+F 1 "PJ398SM" H 5522 5425 50  0000 R CNN
 F 2 "ell_connectors:THONKICONN" H 5983 5633 50  0001 C CNN
 F 3 "" H 6100 5150 50  0000 C CNN
@@
 Connection ~ 5100 5550
 Connection ~ 4300 5550
+Text Notes 3700 1400 0    50   ~ 0
+Audio In L\n
+Text Notes 3700 2750 0    50   ~ 0
+Audio In R\n
+Text Notes 6500 3950 0    50   ~ 0
+Audio Out L\n
+Text Notes 6500 5250 0    50   ~ 0
+Audio Out R
 $EndSCHEMATC
