File: hardware/mainboard/Channel_Buttons_And_Switches.sch (KiCad schematic (older format))
At the start: 20 parts, among them SW10 BTTN_PLAY_B, SW11 BTTN_PLAY_C, SW12 BTTN_PLAY_D, SW5 BTTN_SPEED_A, SW6 BTTN_SPEED_B, SW7 BTTN_SPEED_C, SW8 BTTN_SPEED_D, SW9 BTTN_PLAY_A

Commit message: hardware: update schematics & add BOM
Parts:
- SW10: value BTTN_PLAY_B -> D6R90F1LFS
- SW11: value BTTN_PLAY_C -> D6R90F1LFS
- SW12: value BTTN_PLAY_D -> D6R90F1LFS
- SW5: value BTTN_SPEED_A -> C&K 7105SYCQE
- SW6: value BTTN_SPEED_B -> C&K 7105SYCQE
- SW7: value BTTN_SPEED_C -> C&K 7105SYCQE
- SW8: value BTTN_SPEED_D -> C&K 7105SYCQE
- SW9: value BTTN_PLAY_A -> D6R90F1LFS
Changed lines of the file:
@@
 AR Path="/61F0493E/61F27F8E" Ref="SW9"  Part="1"
 F 0 "SW9" H 10300 1885 50  0000 C CNN
-F 1 "BTTN_PLAY_A" H 10300 1794 50  0000 C CNN
+F 1 "D6R90F1LFS " H 10300 1794 50  0000 C CNN
 F 2 "ell_special:CK-D6R_Pushbutton" H 10300 1650 50  0001 C CNN
 F 3 "~" H 10300 1650 50  0001 C CNN
@@
 AR Path="/61F0493E/61F27FCD" Ref="SW10"  Part="1"
 F 0 "SW10" H 10300 3135 50  0000 C CNN
-F 1 "BTTN_PLAY_B" H 10300 3044 50  0000 C CNN
+F 1 "D6R90F1LFS " H 10300 3044 50  0000 C CNN
 F 2 "ell_special:CK-D6R_Pushbutton" H 10300 2900 50  0001 C CNN
 F 3 "~" H 10300 2900 50  0001 C CNN
@@
 AR Path="/61F0493E/61F27FED" Ref="SW6"  Part="1"
 F 0 "SW6" H 8650 3250 50  0000 C CNN
-F 1 "BTTN_SPEED_B" H 8800 3150 50  0000 C CNN
+F 1 "C&K 7105SYCQE" H 8800 3150 50  0000 C CNN
 F 2 "ell_special:7105SYCQE-1P3T-SP3T-Switch" H 8650 2900 50  0001 C CNN
 F 3 "~" H 8650 2900 50  0001 C CNN
@@
 P 8650 1650
 F 0 "SW5" H 8650 2000 50  0000 C CNN
-F 1 "BTTN_SPEED_A" H 8800 1900 50  0000 C CNN
+F 1 "C&K 7105SYCQE" H 8800 1900 50  0000 C CNN
 F 2 "ell_special:7105SYCQE-1P3T-SP3T-Switch" H 8650 1650 50  0001 C CNN
 F 3 "~" H 8650 1650 50  0001 C CNN
@@
 AR Path="/61F0493E/61F28032" Ref="SW11"  Part="1"
 F 0 "SW11" H 10300 4385 50  0000 C CNN
-F 1 "BTTN_PLAY_C" H 10300 4294 50  0000 C CNN
+F 1 "D6R90F1LFS " H 10300 4294 50  0000 C CNN
 F 2 "ell_special:CK-D6R_Pushbutton" H 10300 4150 50  0001 C CNN
 F 3 "~" H 10300 4150 50  0001 C CNN
@@
 AR Path="/61F0493E/61F28071" Ref="SW12"  Part="1"
 F 0 "SW12" H 10300 5635 50  0000 C CNN
-F 1 "BTTN_PLAY_D" H 10300 5544 50  0000 C CNN
+F 1 "D6R90F1LFS " H 10300 5544 50  0000 C CNN
 F 2 "ell_special:CK-D6R_Pushbutton" H 10300 5400 50  0001 C CNN
 F 3 "~" H 10300 5400 50  0001 C CNN
@@
 AR Path="/61F0493E/61F28091" Ref="SW8"  Part="1"
 F 0 "SW8" H 8650 5750 50  0000 C CNN
-F 1 "BTTN_SPEED_D" H 8800 5650 50  0000 C CNN
+F 1 "C&K 7105SYCQE" H 8800 5650 50  0000 C CNN
 F 2 "ell_special:7105SYCQE-1P3T-SP3T-Switch" H 8650 5400 50  0001 C CNN
 F 3 "~" H 8650 5400 50  0001 C CNN
@@
 AR Path="/61F0493E/61F280C3" Ref="SW7"  Part="1"
 F 0 "SW7" H 8650 4500 50  0000 C CNN
-F 1 "BTTN_SPEED_C" H 8800 4400 50  0000 C CNN
+F 1 "C&K 7105SYCQE" H 8800 4400 50  0000 C CNN
 F 2 "ell_special:7105SYCQE-1P3T-SP3T-Switch" H 8650 4150 50  0001 C CNN
 F 3 "~" H 8650 4150 50  0001 C CNN
