File: hardware/mainboard/Channel_LEDs.sch (KiCad schematic (older format))
At the start: 54 parts, among them U6 PCA9685PW, U7 PCA9685PW

Commit message: hardware: update schematics & add BOM
Parts:
- D12: value LED_SPEED_+2_A -> LED_RED_GREEN_CA
- D13: value LED_SPEED_+2_C -> LED_RED_GREEN_CA
- D14: value LED_SPEED_+1_A -> LED_RED_GREEN_CA
- D15: value LED_SPEED_+1_C -> LED_RED_GREEN_CA
- D16: value LED_SPEED_-1_A -> LED_RED_GREEN_CA
- D17: value LED_SPEED_-1_C -> LED_RED_GREEN_CA
- D18: value LED_SPEED_-2_A -> LED_RED_GREEN_CA
- D19: value LED_SPEED_-2_C -> LED_RED_GREEN_CA
- D20: value LED_SPEED_+2_B -> LED_RED_GREEN_CA
- D21: value LED_SPEED_+2_D -> LED_RED_GREEN_CA
- D22: value LED_SPEED_+1_B -> LED_RED_GREEN_CA
- D23: value LED_SPEED_+1_D -> LED_RED_GREEN_CA
- D24: value LED_SPEED_-1_B -> LED_RED_GREEN_CA
- D25: value LED_SPEED_-1_D -> LED_RED_GREEN_CA
- D26: value LED_SPEED_-2_B -> LED_RED_GREEN_CA
- D27: value LED_SPEED_-2_D -> LED_RED_GREEN_CA
- R39, R40, R41, R42, R43, R44, R45, R46, R47, R48, R49, R50, R51, R52, R53, R54, R55, R56, R57, R58, R59, R60, R61, R62, R63, R64, R65, R66, R67, R68, R69, R70: value Rled -> 330
Other:
- note added: "+1 A"
- note added: "+1 B"
- note added: "+1 C"
- note added: "+1 D"
- note added: "+2 A"
- note added: "+2 B"
- note added: "+2 C"
- note added: "+2 D"
- note added: "-1 A\n"
- note added: "-1 B"
- note added: "-1 C"
- note added: "-1 D"
- note added: "-2 A"
- note added: "-2 B"
- note added: "-2 C\n"
- note added: "-2 D"
