File: hardware/mainboard/Common_LEDs_And_Buttons.sch (KiCad schematic (older format))
At the start: 38 parts, among them SW1 BTTN_LOAD, SW2 BTTN_DIRECTION, SW3 BTTN_SAVE, SW4 BTTN_REC, U5 PCA9685PW

Commit message: hardware: update schematics & add BOM
Parts:
- D10: value LED_DIRECTION -> LED_RED_GREEN_CA
- D11: value LED_REC -> LED_RED_GREEN_CA
- D4: value LED_IN_L -> LED_RED_GREEN_CA
- D5: value LED_IN_R -> LED_RED_GREEN_CA
- D6: value LED_OUT_L -> LED_RED_GREEN_CA
- D7: value LED_OUT_R -> LED_RED_GREEN_CA
- D8: value LED_LOAD -> LED_RED_GREEN_CA
- D9: value LED_SAVE -> LED_RED_GREEN_CA
- R21, R22, R23, R26, R27, R28, R29, R30, R31, R32, R33, R34, R35, R36, R37, R38: value Rled -> 330
- SW1: value BTTN_LOAD -> TL1105SPF250Q
- SW2: value BTTN_DIRECTION -> TL1105SPF250Q
- SW3: value BTTN_SAVE -> TL1105SPF250Q
- SW4: value BTTN_REC -> D6R40F1LFS
Connections:
- net BTTN_DIRECTION renamed BTTN_SETTINGS
Other:
- note added: "In L\n"
- note added: "In R"
- note added: "Load\n"
- note added: "Out L\n"
- note added: "Out R"
- note added: "Rec\n"
- note added: "Save"
- note added: "Settings"
Changed lines of the file:
@@
 AR Path="/61C6F729" Ref="SW?"  Part="1"
 F 0 "SW3" H 5050 6035 50  0000 C CNN
-F 1 "BTTN_SAVE" H 5050 5944 50  0000 C CNN
+F 1 "TL1105SPF250Q" H 5050 5944 50  0000 C CNN
 F 2 "Button_Switch_THT:SW_PUSH_6mm" H 5050 5800 50  0001 C CNN
 F 3 "~" H 5050 5800 50  0001 C CNN
@@
 AR Path="/61C6F749" Ref="SW?"  Part="1"
 F 0 "SW4" H 5050 7035 50  0000 C CNN
-F 1 "BTTN_REC" H 5050 6944 50  0000 C CNN
+F 1 "D6R40F1LFS " H 5050 6944 50  0000 C CNN
 F 2 "ell_special:CK-D6R_Pushbutton" H 5050 6800 50  0001 C CNN
 F 3 "~" H 5050 6800 50  0001 C CNN
@@
 AR Path="/61C6F769" Ref="SW?"  Part="1"
 F 0 "SW1" H 3450 6035 50  0000 C CNN
-F 1 "BTTN_LOAD" H 3450 5944 50  0000 C CNN
+F 1 "TL1105SPF250Q" H 3450 5944 50  0000 C CNN
 F 2 "Button_Switch_THT:SW_PUSH_6mm" H 3450 5800 50  0001 C CNN
 F 3 "~" H 3450 5800 50  0001 C CNN
@@
 AR Path="/61C6F789" Ref="SW?"  Part="1"
 F 0 "SW2" H 3450 7035 50  0000 C CNN
-F 1 "BTTN_DIRECTION" H 3450 6944 50  0000 C CNN
+F 1 "TL1105SPF250Q" H 3450 6944 50  0000 C CNN
 F 2 "Button_Switch_THT:SW_PUSH_6mm" H 3450 6800 50  0001 C CNN
 F 3 "~" H 3450 6800 50  0001 C CNN
@@
 $EndComp
 Text GLabel 2900 6800 0    50   Output ~ 0
-BTTN_DIRECTION
+BTTN_SETTINGS
 $Comp
 L Driver_LED:PCA9685PW U5
@@
 AR Path="/61C6F7D7" Ref="D?"  Part="1"
 F 0 "D4" V 8250 1700 50  0000 L CNN
-F 1 "LED_IN_L" H 9050 1550 50  0000 L CNN
+F 1 "LED_RED_GREEN_CA" H 9050 1550 50  0000 L CNN
 F 2 "LED_THT:LED_D3.0mm-3" H 8500 1550 50  0001 C CNN
 F 3 "~" H 8500 1550 50  0001 C CNN
@@
 AR Path="/61C6F7DD" Ref="R?"  Part="1"
 F 0 "R21" H 8420 2046 50  0000 L CNN
-F 1 "Rled" H 8420 1955 50  0000 L CNN
+F 1 "330" H 8420 1955 50  0000 L CNN
 F 2 "Resistor_SMD:R_0603_1608Metric_Pad0.98x0.95mm_HandSolder" V 8280 2000 50  0001 C CNN
 F 3 "~" H 8350 2000 50  0001 C CNN
@@
 AR Path="/61C6F7E3" Ref="R?"  Part="1"
 F 0 "R22" H 8620 2046 50  0000 L CNN
-F 1 "Rled" H 8620 1955 50  0000 L CNN
+F 1 "330" H 8620 1955 50  0000 L CNN
 F 2 "Resistor_SMD:R_0603_1608Metric_Pad0.98x0.95mm_HandSolder" V 8480 2000 50  0001 C CNN
 F 3 "~" H 8550 2000 50  0001 C CNN
@@
 AR Path="/61C6F7F0" Ref="D?"  Part="1"
 F 0 "D5" V 7700 1700 50  0000 L CNN
-F 1 "LED_IN_R" H 8500 1550 50  0000 L CNN
+F 1 "LED_RED_GREEN_CA" H 8500 1550 50  0000 L CNN
 F 2 "LED_THT:LED_D3.0mm-3" H 7950 1550 50  0001 C CNN
 F 3 "~" H 7950 1550 50  0001 C CNN
@@
 AR Path="/61C6F7F6" Ref="R?"  Part="1"
 F 0 "R23" H 7870 2046 50  0000 L CNN
-F 1 "Rled" H 7870 1955 50  0000 L CNN
+F 1 "330" H 7870 1955 50  0000 L CNN
 F 2 "Resistor_SMD:R_0603_1608Metric_Pad0.98x0.95mm_HandSolder" V 7730 2000 50  0001 C CNN
 F 3 "~" H 7800 2000 50  0001 C CNN
@@
 AR Path="/61C6F7FC" Ref="R?"  Part="1"
 F 0 "R26" H 8070 2046 50  0000 L CNN
-F 1 "Rled" H 8070 1955 50  0000 L CNN
+F 1 "330" H 8070 1955 50  0000 L CNN
 F 2 "Resistor_SMD:R_0603_1608Metric_Pad0.98x0.95mm_HandSolder" V 7930 2000 50  0001 C CNN
 F 3 "~" H 8000 2000 50  0001 C CNN
@@
 AR Path="/61C6F809" Ref="D?"  Part="1"
 F 0 "D6" V 7150 1700 50  0000 L CNN
-F 1 "LED_OUT_L" H 7950 1550 50  0000 L CNN
+F 1 "LED_RED_GREEN_CA" H 7950 1550 50  0000 L CNN
 F 2 "LED_THT:LED_D3.0mm-3" H 7400 1550 50  0001 C CNN
 F 3 "~" H 7400 1550 50  0001 C CNN
@@
 AR Path="/61C6F80F" Ref="R?"  Part="1"
 F 0 "R27" H 7320 2046 50  0000 L CNN
-F 1 "Rled" H 7320 1955 50  0000 L CNN
+F 1 "330" H 7320 1955 50  0000 L CNN
 F 2 "Resistor_SMD:R_0603_1608Metric_Pad0.98x0.95mm_HandSolder" V 7180 2000 50  0001 C CNN
 F 3 "~" H 7250 2000 50  0001 C CNN
@@
 AR Path="/61C6F815" Ref="R?"  Part="1"
 F 0 "R28" H 7520 2046 50  0000 L CNN
-F 1 "Rled" H 7520 1955 50  0000 L CNN
+F 1 "330" H 7520 1955 50  0000 L CNN
 F 2 "Resistor_SMD:R_0603_1608Metric_Pad0.98x0.95mm_HandSolder" V 7380 2000 50  0001 C CNN
 F 3 "~" H 7450 2000 50  0001 C CNN
@@
 AR Path="/61C6F822" Ref="D?"  Part="1"
 F 0 "D7" V 6600 1700 50  0000 L CNN
-F 1 "LED_OUT_R" H 7400 1550 50  0000 L CNN
+F 1 "LED_RED_GREEN_CA" H 7400 1550 50  0000 L CNN
 F 2 "LED_THT:LED_D3.0mm-3" H 6850 1550 50  0001 C CNN
 F 3 "~" H 6850 1550 50  0001 C CNN
@@
 AR Path="/61C6F828" Ref="R?"  Part="1"
 F 0 "R29" H 6770 2046 50  0000 L CNN
-F 1 "Rled" H 6770 1955 50  0000 L CNN
+F 1 "330" H 6770 1955 50  0000 L CNN
 F 2 "Resistor_SMD:R_0603_1608Metric_Pad0.98x0.95mm_HandSolder" V 6630 2000 50  0001 C CNN
 F 3 "~" H 6700 2000 50  0001 C CNN
@@
 AR Path="/61C6F82E" Ref="R?"  Part="1"
 F 0 "R30" H 6970 2046 50  0000 L CNN
-F 1 "Rled" H 6970 1955 50  0000 L CNN
+F 1 "330" H 6970 1955 50  0000 L CNN
 F 2 "Resistor_SMD:R_0603_1608Metric_Pad0.98x0.95mm_HandSolder" V 6830 2000 50  0001 C CNN
 F 3 "~" H 6900 2000 50  0001 C CNN
@@
 	4800 2700 3900 2700
 $Comp
-L Device:LED_Dual_CAC D8
-U 1 1 61C6F843
-P 4700 1550
-AR Path="/61A6EF5C/61C6F843" Ref="D8"  Part="1"
-AR Path="/61C6F843" Ref="D?"  Part="1"
-F 0 "D8" V 4500 1700 50  0000 L CNN
-F 1 "LED_LOAD" H 5300 1550 50  0000 L CNN
-F 2 "LED_THT:LED_D3.0mm-3" H 4750 1550 50  0001 C CNN
-F 3 "~" H 4750 1550 50  0001 C CNN
-	1    4700 1550
-	0    1    1    0
-$EndComp
-$Comp
 L Device:R R31
 U 1 1 61C6F849
@@
 AR Path="/61C6F849" Ref="R?"  Part="1"
 F 0 "R31" H 4670 2046 50  0000 L CNN
-F 1 "Rled" H 4670 1955 50  0000 L CNN
+F 1 "330" H 4670 1955 50  0000 L CNN
 F 2 "Resistor_SMD:R_0603_1608Metric_Pad0.98x0.95mm_HandSolder" V 4530 2000 50  0001 C CNN
 F 3 "~" H 4600 2000 50  0001 C CNN
@@
 AR Path="/61C6F84F" Ref="R?"  Part="1"
 F 0 "R32" H 4870 2046 50  0000 L CNN
-F 1 "Rled" H 4870 1955 50  0000 L CNN
+F 1 "330" H 4870 1955 50  0000 L CNN
 F 2 "Resistor_SMD:R_0603_1608Metric_Pad0.98x0.95mm_HandSolder" V 4730 2000 50  0001 C CNN
 F 3 "~" H 4800 2000 50  0001 C CNN
@@
 AR Path="/61C93593" Ref="D?"  Part="1"
 F 0 "D9" V 5300 1700 50  0000 L CNN
-F 1 "LED_SAVE" H 6100 1550 50  0000 L CNN
+F 1 "LED_RED_GREEN_CA" H 6100 1550 50  0000 L CNN
 F 2 "LED_THT:LED_D3.0mm-3" H 5550 1550 50  0001 C CNN
 F 3 "~" H 5550 1550 50  0001 C CNN
@@
 AR Path="/61C93599" Ref="R?"  Part="1"
 F 0 "R33" H 5470 2046 50  0000 L CNN
-F 1 "Rled" H 5470 1955 50  0000 L CNN
+F 1 "330" H 5470 1955 50  0000 L CNN
 F 2 "Resistor_SMD:R_0603_1608Metric_Pad0.98x0.95mm_HandSolder" V 5330 2000 50  0001 C CNN
 F 3 "~" H 5400 2000 50  0001 C CNN
@@
 AR Path="/61C9359F" Ref="R?"  Part="1"
 F 0 "R34" H 5670 2046 50  0000 L CNN
-F 1 "Rled" H 5670 1955 50  0000 L CNN
+F 1 "330" H 5670 1955 50  0000 L CNN
 F 2 "Resistor_SMD:R_0603_1608Metric_Pad0.98x0.95mm_HandSolder" V 5530 2000 50  0001 C CNN
 F 3 "~" H 5600 2000 50  0001 C CNN
@@
 AR Path="/61C96285" Ref="D?"  Part="1"
 F 0 "D10" V 5850 1700 50  0000 L CNN
-F 1 "LED_DIRECTION" H 6650 1550 50  0000 L CNN
+F 1 "LED_RED_GREEN_CA" H 6650 1550 50  0000 L CNN
 F 2 "LED_THT:LED_D3.0mm-3" H 6100 1550 50  0001 C CNN
 F 3 "~" H 6100 1550 50  0001 C CNN
@@
 AR Path="/61C9628B" Ref="R?"  Part="1"
 F 0 "R35" H 6020 2046 50  0000 L CNN
-F 1 "Rled" H 6020 1955 50  0000 L CNN
+F 1 "330" H 6020 1955 50  0000 L CNN
 F 2 "Resistor_SMD:R_0603_1608Metric_Pad0.98x0.95mm_HandSolder" V 5880 2000 50  0001 C CNN
 F 3 "~" H 5950 2000 50  0001 C CNN
@@
 AR Path="/61C96291" Ref="R?"  Part="1"
 F 0 "R36" H 6220 2046 50  0000 L CNN
-F 1 "Rled" H 6220 1955 50  0000 L CNN
+F 1 "330" H 6220 1955 50  0000 L CNN
 F 2 "Resistor_SMD:R_0603_1608Metric_Pad0.98x0.95mm_HandSolder" V 6080 2000 50  0001 C CNN
 F 3 "~" H 6150 2000 50  0001 C CNN
@@
 AR Path="/61C99EF2" Ref="D?"  Part="1"
 F 0 "D11" V 3950 1700 50  0000 L CNN
-F 1 "LED_REC" H 4750 1550 50  0000 L CNN
+F 1 "LED_RED_GREEN_CA" H 4750 1550 50  0000 L CNN
 F 2 "LED_THT:LED_D3.0mm-3" H 4200 1550 50  0001 C CNN
 F 3 "~" H 4200 1550 50  0001 C CNN
@@
 AR Path="/61C99EF8" Ref="R?"  Part="1"
 F 0 "R37" H 4120 2046 50  0000 L CNN
-F 1 "Rled" H 4120 1955 50  0000 L CNN
+F 1 "330" H 4120 1955 50  0000 L CNN
 F 2 "Resistor_SMD:R_0603_1608Metric_Pad0.98x0.95mm_HandSolder" V 3980 2000 50  0001 C CNN
 F 3 "~" H 4050 2000 50  0001 C CNN
@@
 AR Path="/61C99EFE" Ref="R?"  Part="1"
 F 0 "R38" H 4320 2046 50  0000 L CNN
-F 1 "Rled" H 4320 1955 50  0000 L CNN
+F 1 "330" H 4320 1955 50  0000 L CNN
 F 2 "Resistor_SMD:R_0603_1608Metric_Pad0.98x0.95mm_HandSolder" V 4180 2000 50  0001 C CNN
 F 3 "~" H 4250 2000 50  0001 C CNN
@@
 Wire Wire Line
 	2250 3400 2250 3300
+$Comp
+L Device:LED_Dual_CAC D8
+U 1 1 61C6F843
+P 4700 1550
+AR Path="/61A6EF5C/61C6F843" Ref="D8"  Part="1"
+AR Path="/61C6F843" Ref="D?"  Part="1"
+F 0 "D8" V 4500 1700 50  0000 L CNN
+F 1 "LED_RED_GREEN_CA" H 5300 1550 50  0000 L CNN
+F 2 "LED_THT:LED_D3.0mm-3" H 4750 1550 50  0001 C CNN
+F 3 "~" H 4750 1550 50  0001 C CNN
+	1    4700 1550
+	0    1    1    0
+$EndComp
+Text Notes 4100 850  0    50   ~ 0
+Rec\n
+Text Notes 4600 850  0    50   ~ 0
+Load\n
+Text Notes 5400 850  0    50   ~ 0
+Save
+Text Notes 5900 850  0    50   ~ 0
+Settings
+Text Notes 6700 850  0    50   ~ 0
+Out R
+Text Notes 7250 850  0    50   ~ 0
+Out L\n
+Text Notes 7800 850  0    50   ~ 0
+In R
+Text Notes 8350 850  0    50   ~ 0
+In L\n
 $EndSCHEMATC
