File: hardware/mainboard/LEDs.sch (KiCad schematic (older format))
At the start: 74 parts

Commit message: hardware: update schematics & add BOM
Parts:
- D?: value LED_SPEED_+2_A -> LED_RED_GREEN_CA
- D?: value LED_SPEED_+1_A -> LED_RED_GREEN_CA
- D?: value LED_SPEED_-1_A -> LED_RED_GREEN_CA
- D?: value LED_SPEED_-2_A -> LED_RED_GREEN_CA
- D?: value LED_SPEED_+2_B -> LED_RED_GREEN_CA
- D?: value LED_SPEED_+1_B -> LED_RED_GREEN_CA
- D?: value LED_SPEED_-1_B -> LED_RED_GREEN_CA
- D?: value LED_SPEED_-2_B -> LED_RED_GREEN_CA
- D?: value LED_SPEED_+2_C -> LED_RED_GREEN_CA
- D?: value LED_SPEED_+1_C -> LED_RED_GREEN_CA
- D?: value LED_SPEED_-1_C -> LED_RED_GREEN_CA
- D?: value LED_SPEED_-2_C -> LED_RED_GREEN_CA
- D?: value LED_SPEED_+2_D -> LED_RED_GREEN_CA
- D?: value LED_SPEED_+1_D -> LED_RED_GREEN_CA
- D?: value LED_SPEED_-1_D -> LED_RED_GREEN_CA
- D?: value LED_SPEED_-2_D -> LED_RED_GREEN_CA
- R? (x32): value Rled -> 330
