File: hardware/mainboard/UI.sch (KiCad schematic (older format))
At the start: 38 parts, among them SW1 BTTN_LOAD, SW2 BTTN_DIRECTION, SW3 BTTN_SAVE, SW4 BTTN_REC, U7 PCA9685PW

Commit message: hardware: update schematics & add BOM
Parts:
- R19, R20, R21, R22, R23, R26, R27, R28, R29, R30, R33, R34, R35, R36, R37, R38: value Rled -> 330
Changed lines of the file:
@@
 AR Path="/61C6F7DD" Ref="R?"  Part="1"
 F 0 "R19" H 4120 2046 50  0000 L CNN
-F 1 "Rled" H 4120 1955 50  0000 L CNN
+F 1 "330" H 4120 1955 50  0000 L CNN
 F 2 "Resistor_SMD:R_0603_1608Metric_Pad0.98x0.95mm_HandSolder" V 3980 2000 50  0001 C CNN
 F 3 "~" H 4050 2000 50  0001 C CNN
@@
 AR Path="/61C6F7E3" Ref="R?"  Part="1"
 F 0 "R20" H 4320 2046 50  0000 L CNN
-F 1 "Rled" H 4320 1955 50  0000 L CNN
+F 1 "330" H 4320 1955 50  0000 L CNN
 F 2 "Resistor_SMD:R_0603_1608Metric_Pad0.98x0.95mm_HandSolder" V 4180 2000 50  0001 C CNN
 F 3 "~" H 4250 2000 50  0001 C CNN
@@
 AR Path="/61C6F7F6" Ref="R?"  Part="1"
 F 0 "R21" H 4670 2046 50  0000 L CNN
-F 1 "Rled" H 4670 1955 50  0000 L CNN
+F 1 "330" H 4670 1955 50  0000 L CNN
 F 2 "Resistor_SMD:R_0603_1608Metric_Pad0.98x0.95mm_HandSolder" V 4530 2000 50  0001 C CNN
 F 3 "~" H 4600 2000 50  0001 C CNN
@@
 AR Path="/61C6F7FC" Ref="R?"  Part="1"
 F 0 "R22" H 4870 2046 50  0000 L CNN
-F 1 "Rled" H 4870 1955 50  0000 L CNN
+F 1 "330" H 4870 1955 50  0000 L CNN
 F 2 "Resistor_SMD:R_0603_1608Metric_Pad0.98x0.95mm_HandSolder" V 4730 2000 50  0001 C CNN
 F 3 "~" H 4800 2000 50  0001 C CNN
@@
 AR Path="/61C6F80F" Ref="R?"  Part="1"
 F 0 "R23" H 5470 2046 50  0000 L CNN
-F 1 "Rled" H 5470 1955 50  0000 L CNN
+F 1 "330" H 5470 1955 50  0000 L CNN
 F 2 "Resistor_SMD:R_0603_1608Metric_Pad0.98x0.95mm_HandSolder" V 5330 2000 50  0001 C CNN
 F 3 "~" H 5400 2000 50  0001 C CNN
@@
 AR Path="/61C6F815" Ref="R?"  Part="1"
 F 0 "R26" H 5670 2046 50  0000 L CNN
-F 1 "Rled" H 5670 1955 50  0000 L CNN
+F 1 "330" H 5670 1955 50  0000 L CNN
 F 2 "Resistor_SMD:R_0603_1608Metric_Pad0.98x0.95mm_HandSolder" V 5530 2000 50  0001 C CNN
 F 3 "~" H 5600 2000 50  0001 C CNN
@@
 AR Path="/61C6F828" Ref="R?"  Part="1"
 F 0 "R27" H 6020 2046 50  0000 L CNN
-F 1 "Rled" H 6020 1955 50  0000 L CNN
+F 1 "330" H 6020 1955 50  0000 L CNN
 F 2 "Resistor_SMD:R_0603_1608Metric_Pad0.98x0.95mm_HandSolder" V 5880 2000 50  0001 C CNN
 F 3 "~" H 5950 2000 50  0001 C CNN
@@
 AR Path="/61C6F82E" Ref="R?"  Part="1"
 F 0 "R28" H 6220 2046 50  0000 L CNN
-F 1 "Rled" H 6220 1955 50  0000 L CNN
+F 1 "330" H 6220 1955 50  0000 L CNN
 F 2 "Resistor_SMD:R_0603_1608Metric_Pad0.98x0.95mm_HandSolder" V 6080 2000 50  0001 C CNN
 F 3 "~" H 6150 2000 50  0001 C CNN
@@
 AR Path="/61C6F849" Ref="R?"  Part="1"
 F 0 "R29" H 6770 2046 50  0000 L CNN
-F 1 "Rled" H 6770 1955 50  0000 L CNN
+F 1 "330" H 6770 1955 50  0000 L CNN
 F 2 "Resistor_SMD:R_0603_1608Metric_Pad0.98x0.95mm_HandSolder" V 6630 2000 50  0001 C CNN
 F 3 "~" H 6700 2000 50  0001 C CNN
@@
 AR Path="/61C6F84F" Ref="R?"  Part="1"
 F 0 "R30" H 6970 2046 50  0000 L CNN
-F 1 "Rled" H 6970 1955 50  0000 L CNN
+F 1 "330" H 6970 1955 50  0000 L CNN
 F 2 "Resistor_SMD:R_0603_1608Metric_Pad0.98x0.95mm_HandSolder" V 6830 2000 50  0001 C CNN
 F 3 "~" H 6900 2000 50  0001 C CNN
@@
 AR Path="/61C93599" Ref="R?"  Part="1"
 F 0 "R33" H 7320 2046 50  0000 L CNN
-F 1 "Rled" H 7320 1955 50  0000 L CNN
+F 1 "330" H 7320 1955 50  0000 L CNN
 F 2 "Resistor_SMD:R_0603_1608Metric_Pad0.98x0.95mm_HandSolder" V 7180 2000 50  0001 C CNN
 F 3 "~" H 7250 2000 50  0001 C CNN
@@
 AR Path="/61C9359F" Ref="R?"  Part="1"
 F 0 "R34" H 7520 2046 50  0000 L CNN
-F 1 "Rled" H 7520 1955 50  0000 L CNN
+F 1 "330" H 7520 1955 50  0000 L CNN
 F 2 "Resistor_SMD:R_0603_1608Metric_Pad0.98x0.95mm_HandSolder" V 7380 2000 50  0001 C CNN
 F 3 "~" H 7450 2000 50  0001 C CNN
@@
 AR Path="/61C9628B" Ref="R?"  Part="1"
 F 0 "R35" H 7870 2046 50  0000 L CNN
-F 1 "Rled" H 7870 1955 50  0000 L CNN
+F 1 "330" H 7870 1955 50  0000 L CNN
 F 2 "Resistor_SMD:R_0603_1608Metric_Pad0.98x0.95mm_HandSolder" V 7730 2000 50  0001 C CNN
 F 3 "~" H 7800 2000 50  0001 C CNN
@@
 AR Path="/61C96291" Ref="R?"  Part="1"
 F 0 "R36" H 8070 2046 50  0000 L CNN
-F 1 "Rled" H 8070 1955 50  0000 L CNN
+F 1 "330" H 8070 1955 50  0000 L CNN
 F 2 "Resistor_SMD:R_0603_1608Metric_Pad0.98x0.95mm_HandSolder" V 7930 2000 50  0001 C CNN
 F 3 "~" H 8000 2000 50  0001 C CNN
@@
 AR Path="/61C99EF8" Ref="R?"  Part="1"
 F 0 "R37" H 8420 2046 50  0000 L CNN
-F 1 "Rled" H 8420 1955 50  0000 L CNN
+F 1 "330" H 8420 1955 50  0000 L CNN
 F 2 "Resistor_SMD:R_0603_1608Metric_Pad0.98x0.95mm_HandSolder" V 8280 2000 50  0001 C CNN
 F 3 "~" H 8350 2000 50  0001 C CNN
@@
 AR Path="/61C99EFE" Ref="R?"  Part="1"
 F 0 "R38" H 8620 2046 50  0000 L CNN
-F 1 "Rled" H 8620 1955 50  0000 L CNN
+F 1 "330" H 8620 1955 50  0000 L CNN
 F 2 "Resistor_SMD:R_0603_1608Metric_Pad0.98x0.95mm_HandSolder" V 8480 2000 50  0001 C CNN
 F 3 "~" H 8550 2000 50  0001 C CNN
