File: hardware/mainboard/AudioIO.kicad_sch (KiCad schematic)
At the start: 25 parts, among them J701 PJ398SM, J702 PJ398SM, J703 PJ398SM, J704 PJ398SM

Commit message: hardware: resave files with KiCad v7.0.4
Parts:
- gave numbers to parts that had none: 17
Connections:
- net AUDIO_ADC_L: now also U701.8; no longer U701.1
- net AUDIO_ADC_R: now also U701.14; no longer U701.1
- net GNDA: now also U701.10 (+), U701.12 (+), U701.5 (+); no longer U701.3 (+), U701.3 (+), U701.3 (+)
- net at C701.2, R701.1, R702.2: now also U701.9 (-); no longer U701.2 (-)
- net at C703.2, R703.1, R704.2: now also U701.13 (-); no longer U701.2 (-)
- net at C705.1, R705.2, R707.1: now also U701.7; no longer U701.1
- net at C705.2, R706.1, R707.2: now also U701.6 (-); no longer U701.2 (-)

Commit message: hardware: change audio I/O gain slightly
Parts:
- R702, R704, R706, R709: value 10k -> 8k2
Changed lines of the file:
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@@
 			)
 		)
-		(property "Value" "10k"
+		(property "Value" "8k2"
 			(at 146.05 48.26 90)
 			(effects
@@
 			)
 		)
-		(property "Value" "10k"
+		(property "Value" "8k2"
 			(at 146.05 82.55 90)
 			(effects
@@
 			)
 		)
-		(property "Value" "10k"
+		(property "Value" "8k2"
 			(at 102.87 107.95 90)
 			(effects
@@
 			)
 		)
-		(property "Value" "10k"
+		(property "Value" "8k2"
 			(at 102.87 140.97 90)
 			(effects
