File: hardware/mainboard/Channel_Buttons_And_Switches.kicad_sch (KiCad schematic)
At the start: 20 parts, among them SW301 C&K 7105SYCQE

Commit message: hardware: resave files with KiCad v7.0.4
Parts:
- SW302, SW304, SW306, SW308: renamed from SW?; value D6R90F1LFS -> D6R90F1LFS
- gave numbers to parts that had none: 15
