File: hardware/mainboard/Channel_Pots_And_Sliders.kicad_sch (KiCad schematic)
At the start: 20 parts

Commit message: hardware: resave files with KiCad v7.0.4
Parts:
- renumbered RV2 to RV505, RV7 to RV506, RV12 to RV507, RV17 to RV508
