File: hardware/mainboard/Common_LEDs_And_Buttons.kicad_sch (KiCad schematic)
At the start: 38 parts

Commit message: hardware: resave files with KiCad v7.0.4
Parts:
- SW204: renamed from SW?; value D6R40F1LFS -> D6R40F1LFS
- gave numbers to parts that had none: 37
