File: hardware/mainboard/Power.kicad_sch (KiCad schematic)
At the start: 26 parts, among them U801 LM4040DBZ-5, U802 AZ1117-3.3, U803 LM4040DBZ-10

Commit message: hardware: resave files with KiCad v7.0.4
Parts:
- gave numbers to parts that had none: 17
